File: BME680_shield.kicad_sch (KiCad schematic)
At the start: 19 parts, among them J101 Conn_01x06, J102 Conn_01x02_Socket, U101 BME680, U102 ESP8266_WeMos_D1_mini, U103 AP7361C-33E, U104 MAX1811

Commit message: push after order
Parts:
- added C103: 10µ, Capacitor_SMD:C_0805_2012Metric_Pad1.18x1.45mm_HandSolder, symbol Device:C
Connections:
- net +3V3: now also C103.1
- net GND: now also C103.2
- net SDA: now reaches J101.4 (Pin_4), R103.2, U101.3 (SDI), U102.13 (D2)
- net SCL: now reaches J101.3 (Pin_3), R102.2, U101.4 (SCK), U102.14 (D1)
Other:
- moved on the sheet: C101, C102, J101, JP101, JP102, JP103, R101, R102, R103, R104, R105, U101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
