File: BME680_shield.kicad_pcb (KiCad board)
At the start: 2 copper layers, 42.5 x 27 mm, 19 parts, among them J101 Conn_01x06, J102 Conn_01x02_Socket, U101 BME680, U102 ESP8266_WeMos_D1_mini, U103 AP7361C-33E, U104 MAX1811

Commit message: push after order
Parts:
- added C103: 10µ, Capacitor_SMD:C_0805_2012Metric_Pad1.18x1.45mm_HandSolder, F.Cu at (108.0, 71.5)
Routing:
- net Net-(U102-A0): track 17.1 -> 15.1 mm
- net GND: track 28.6 -> 28.7 mm, vias 15 -> 19
Other:
- board size 42.5 x 27 mm -> 36.5 x 27 mm
- board text added: "+"
- board text added: "-"
- board text added: "BME680 ESP8266 D1 mini shield with a 1S Li charger 04/2023 Johannes Rothe GitHub: josero360"
- board text added: "Batt"
- board text added: "SCL"
- board text added: "SDA"
- board text removed: "GND"
- board text removed: "UBatt"

Commit message: Leiterpaltte aufgebaut
Parts:
- moved C101 0.50 mm to (96.8, 69.0)
- moved U101 0.50 mm to (93.3, 69.0)
Routing:
- net GND: track 28.7 -> 28.4 mm, vias 19 -> 18
Other:
- outline, holes or cut-outs redrawn
